File: blinkenrocket_cr2032.brd (EAGLE design)
At the start: 96.3 x 47 mm, 22 parts, among them SW1 SWITCH-4POMRON-6-6-SWITCH, SW2 SWITCH-4POMRON-6-6-SWITCH, U2 EEPROM-I2CEIAJ

Commit message: make the audio signal more straight to reduce the antenna effect
Routing:
- net AVR_AUDIO_IN: track 65.4 -> 43.9 mm
- net E3: track 39.6 -> 46.0 mm, vias 2 -> 1
- net R6/SCK: track 78.2 -> 72.7 mm
- net C1: track 21.0 -> 23.7 mm, vias 1 -> 2
- net B1: track 86.4 -> 85.2 mm
